File: KiCad Circuits/EEE3088F PCB/EEE3088F_V1.0/EEE3088F_V1.0.kicad_pcb (KiCad board)
At the start: 2 copper layers, 60 x 82 mm, 58 parts, among them J1 Conn_01x02_Pin, J2 Conn_02x16_Odd_Even, U1 MT3608, U10 HX SS12D10G6-WJ, U11 HUSB237-AA001-DN06R, U2 INA219AxD, U3 DRV8833PWP, U4 AP2112K-3.3, U5 DRV8833PWP, U6 BQ24074RGT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

Commit message: Updated PCB
Parts:
- added REF**: MountingHole_3.2mm_M3, MountingHole:MountingHole_3.2mm_M3, F.Cu at (90.8, 197.6)
Other:
- board size 60 x 82 mm -> 60 x 70.5 mm
- board text added: "Group Number 23 NGRMAR007 LNGJAM012"

Commit message: added test points
Parts:
- added BAT: TestPoint, TestPoint:TestPoint_Pad_4.0x4.0mm, B.Cu at (95.5, 221.3)
- added BOUT2: TestPoint_2Pole, TestPoint:TestPoint_Bridge_Pitch5.08mm_Drill1.3mm, F.Cu at (72.9, 208.3)
- added IN: TestPoint, TestPoint:TestPoint_Pad_4.0x4.0mm, B.Cu at (71.1, 229.8)
- added IN: TestPoint, TestPoint:TestPoint_Pad_4.0x4.0mm, B.Cu at (93.8, 205.9)
- added IN+: TestPoint, TestPoint:TestPoint_Pad_4.0x4.0mm, B.Cu at (71.7, 236.1)
- added IN-: TestPoint, TestPoint:TestPoint_Pad_4.0x4.0mm, B.Cu at (87.2, 230.7)
- added OUT: TestPoint_2Pole, TestPoint:TestPoint_Bridge_Pitch5.08mm_Drill1.3mm, F.Cu at (66.7, 224.1)
- added TP18: TestPoint_2Pole, TestPoint:TestPoint_Bridge_Pitch5.08mm_Drill1.3mm, F.Cu at (108.0, 206.7)
- added USB HV: TestPoint, TestPoint:TestPoint_Pad_4.0x4.0mm, B.Cu at (67.6, 251.4)
- added VRB IN: TestPoint, TestPoint:TestPoint_Pad_4.0x4.0mm, B.Cu at (108.2, 227.7)
- added VRB OUT: TestPoint, TestPoint:TestPoint_Pad_4.0x4.0mm, B.Cu at (114.1, 224.8)
- added VRL OUT: TestPoint, TestPoint:TestPoint_Pad_4.0x4.0mm, B.Cu at (112.8, 237.3)
- added Vs: TestPoint, TestPoint:TestPoint_Pad_4.0x4.0mm, B.Cu at (80.5, 250.2)
Connections:
- U3 pad : GND -> (no net)
- U5 pad : GND -> (no net)
Routing:
- net GND: track 215.1 -> 217.8 mm

Commit message: Final PCB
Parts:
- removed BOUT2, OUT, TP18: TestPoint_2Pole, TestPoint:TestPoint_Bridge_Pitch5.08mm_Drill1.3mm
- removed IN: TestPoint, TestPoint:TestPoint_Pad_4.0x4.0mm
- TP1: renamed from VRB IN; moved to F.Cu
- TP12: renamed from USB HV
- TP2: renamed from VRB OUT; moved to F.Cu
- TP4: renamed from VRL OUT; moved to F.Cu
- TP5: renamed from IN+; moved to F.Cu
- TP8: renamed from IN; moved to F.Cu
- TP9: renamed from BAT; moved to F.Cu
- moved TP5 30.9 mm to (79.0, 206.0), turned to 180 degrees
- moved TP6 24.6 mm to (74.0, 251.5)
- moved TP7 24.4 mm to (70.5, 228.0)
- moved TP2 24.3 mm to (104.5, 202.5), turned to -90 degrees
- moved TP9 21.3 mm to (85.5, 202.5), turned to 180 degrees
- moved TP1 21.2 mm to (114.5, 248.0), turned to 180 degrees
- moved TP4 18.1 mm to (101.5, 251.5), turned to 180 degrees
- moved TP8 3.34 mm to (95.5, 203.0), turned to 180 degrees
- renumbered IN- to TP6, Vs to TP7
Connections:
- U3 pad : (no net) -> GND
- U5 pad : (no net) -> GND
Routing:
- net 5V Out: track 136.0 -> 176.5 mm, vias 2 -> 4
- net Battery Out: track 141.1 -> 175.9 mm
- net 3.3V Out: track 3.19 -> 35.7 mm, vias 0 -> 5
- net 3V3 Out: track 25.7 -> 57.4 mm
- net Battery: track 73.1 -> 102.9 mm, vias 2 -> 4
- net MOTOR3_B_OUT: track 30.7 -> 57.7 mm, vias 0 -> 3
- net HV: track 98.9 -> 108.9 mm
- net GND: track 217.8 -> 218.4 mm, vias 8 -> 9
- net I2C1_SDA: vias 0 -> 1
